File: hardware/ftdi.sch (KiCad schematic (older format))
At the start: 34 parts, among them U1 FT2232HL-REEL, U2 93LCxxC, Y1 12MHz

Commit message: tidying
Parts:
- R6, R7, R9: Mfg PN CRCW060310K0FKEA -> CRCW060310K0FKEA
Changed lines of the file:
@@
 F 4 "1%, 100mW" V 8700 5000 60  0001 C CNN "Desc"
 F 5 "Vishay" V 8700 5000 60  0001 C CNN "Mfg"
-F 6 "CRCW060310K0FKEA " V 8700 5000 60  0001 C CNN "Mfg PN"
+F 6 "CRCW060310K0FKEA" V 8700 5000 60  0001 C CNN "Mfg PN"
 F 7 "Digikey" V 8700 5000 60  0001 C CNN "Supplier"
 F 8 "541-10.0KHTR-ND" V 8700 5000 60  0001 C CNN "Supplier PN"
@@
 F 4 "1%, 100mW" V 9900 5000 60  0001 C CNN "Desc"
 F 5 "Vishay" V 9900 5000 60  0001 C CNN "Mfg"
-F 6 "CRCW060310K0FKEA " V 9900 5000 60  0001 C CNN "Mfg PN"
+F 6 "CRCW060310K0FKEA" V 9900 5000 60  0001 C CNN "Mfg PN"
 F 7 "Digikey" V 9900 5000 60  0001 C CNN "Supplier"
 F 8 "541-10.0KHTR-ND" V 9900 5000 60  0001 C CNN "Supplier PN"
@@
 F 4 "1%, 100mW" V 10100 5000 60  0001 C CNN "Desc"
 F 5 "Vishay" V 10100 5000 60  0001 C CNN "Mfg"
-F 6 "CRCW060310K0FKEA " V 10100 5000 60  0001 C CNN "Mfg PN"
+F 6 "CRCW060310K0FKEA" V 10100 5000 60  0001 C CNN "Mfg PN"
 F 7 "Digikey" V 10100 5000 60  0001 C CNN "Supplier"
 F 8 "541-10.0KHTR-ND" V 10100 5000 60  0001 C CNN "Supplier PN"
