File: hardware/phy.sch (KiCad schematic (older format))
At the start: 30 parts, among them U10 ACM2012E-T00, U4 DP83822, U5 ALT3232M, U7 ACM2012E-T00, U8 ALT3232M, Y2 25MHz

Commit message: tidying
Parts:
- R12, R15: Mfg PN RCS060375R0FKEA -> RCS060375R0FKEA
Changed lines of the file:
@@
 F 4 "1%, 250mW" V 6400 4600 60  0001 C CNN "Desc"
 F 5 "Vishay" V 6400 4600 60  0001 C CNN "Mfg"
-F 6 " RCS060375R0FKEA " V 6400 4600 60  0001 C CNN "Mfg PN"
+F 6 "RCS060375R0FKEA" V 6400 4600 60  0001 C CNN "Mfg PN"
 F 7 "Digikey" V 6400 4600 60  0001 C CNN "Supplier"
 F 8 "541-2785-1-ND" V 6400 4600 60  0001 C CNN "Supplier PN"
@@
 F 4 "1%, 250mW" V 6600 4600 60  0001 C CNN "Desc"
 F 5 "Vishay" V 6600 4600 60  0001 C CNN "Mfg"
-F 6 " RCS060375R0FKEA " V 6600 4600 60  0001 C CNN "Mfg PN"
+F 6 "RCS060375R0FKEA" V 6600 4600 60  0001 C CNN "Mfg PN"
 F 7 "Digikey" V 6600 4600 60  0001 C CNN "Supplier"
 F 8 "541-2785-1-ND" V 6600 4600 60  0001 C CNN "Supplier PN"
